Commit message: lowering camera and lidar postion

File: notspot_sim_py/src/notspot_description/urdf/camera.xacro (robot description, xacro)
@@ -4,5 +4,5 @@
         <parent link="base_link"/>
         <child link="camera_link"/>
-        <origin xyz="0.276 0 0.181" rpy="0 0.18 0"/>
+        <origin xyz="0.276 0 0.08" rpy="0 0.18 0"/><!--old values:  xyz="0.276 0 0.181" rpy="0 0.18 0"-->
     </joint>
     <link name="camera_link">

File: notspot_sim_py/src/notspot_description/urdf/lidar.xacro (robot description, xacro)
@@ -4,5 +4,5 @@
         <parent link="base_link"/>
         <child link="laser_frame"/>
-        <origin xyz="0.122 0 0.212" rpy="0 0 0"/>
+        lidar: <origin xyz="0.122 0 0.07" rpy="0 0 0"/> <!--<origin xyz="0.122 0 0.212" rpy="0 0 0"/>-->
     </joint>
     <link name="laser_frame">

Commit message: new values for camera and lidar position

File: notspot_sim_py/src/notspot_description/urdf/camera.xacro (robot description, xacro)
@@ -4,5 +4,5 @@
         <parent link="base_link"/>
         <child link="camera_link"/>
-        <origin xyz="0.276 0 0.08" rpy="0 0.18 0"/><!--old values:  xyz="0.276 0 0.181" rpy="0 0.18 0"-->
+        <origin xyz="0.200 0 0.1" rpy="0 0.18 0"/><!--old values:  xyz="0.276 0 0.181" rpy="0 0.18 0"-->
     </joint>
     <link name="camera_link">

File: notspot_sim_py/src/notspot_description/urdf/lidar.xacro (robot description, xacro)
@@ -4,5 +4,5 @@
         <parent link="base_link"/>
         <child link="laser_frame"/>
-        lidar: <origin xyz="0.122 0 0.07" rpy="0 0 0"/> <!--<origin xyz="0.122 0 0.212" rpy="0 0 0"/>-->
+        lidar: <origin xyz="0.046 0 0.1" rpy="0 0 0"/> <!--<origin xyz="0.122 0 0.212" rpy="0 0 0"/>-->
     </joint>
     <link name="laser_frame">

Commit message: another set of new positions for lidar and camera

File: notspot_sim_py/src/notspot_description/urdf/camera.xacro (robot description, xacro)
@@ -4,5 +4,5 @@
         <parent link="base_link"/>
         <child link="camera_link"/>
-        <origin xyz="0.200 0 0.1" rpy="0 0.18 0"/><!--old values:  xyz="0.276 0 0.181" rpy="0 0.18 0"-->
+        <origin xyz="0.14 0 0.11" rpy="0 0.18 0"/><!--old values:  xyz="0.276 0 0.181" rpy="0 0.18 0"-->
     </joint>
     <link name="camera_link">

File: notspot_sim_py/src/notspot_description/urdf/lidar.xacro (robot description, xacro)
@@ -4,5 +4,5 @@
         <parent link="base_link"/>
         <child link="laser_frame"/>
-        lidar: <origin xyz="0.046 0 0.1" rpy="0 0 0"/> <!--<origin xyz="0.122 0 0.212" rpy="0 0 0"/>-->
+        lidar: <origin xyz="-0.014 0 0.11" rpy="0 0 0"/> <!--<origin xyz="0.122 0 0.212" rpy="0 0 0"/>-->
     </joint>
     <link name="laser_frame">
