Commit message: remove 'lidar:' from lidar.xacro

File: notspot_sim_py/src/notspot_description/urdf/lidar.xacro (robot description, xacro)
@@ -4,5 +4,5 @@
         <parent link="base_link"/>
         <child link="laser_frame"/>
-        lidar: <origin xyz="-0.014 0 0.11" rpy="0 0 0"/> <!--<origin xyz="0.122 0 0.212" rpy="0 0 0"/>-->
+        <origin xyz="-0.014 0 0.11" rpy="0 0 0"/> <!--<origin xyz="0.122 0 0.212" rpy="0 0 0"/>-->
     </joint>
     <link name="laser_frame">
